Commit message: ur3e trolley mesh in planning scene, robot repositioned on trolley top
Co-Authored-By: Claude Sonnet 4.6 <noreply@anthropic.com>

File: urdf/ur3e_workcell.urdf.xacro (robot description, xacro)
@@ -12,5 +12,5 @@
     <parent link="world"/>
     <child link="table_mount"/>
-    <origin xyz="0.365 0.355 1.0" rpy="0 0 0"/>
+    <origin xyz="0.23 -0.03 0.724" rpy="0 0 0"/>
   </joint>
   <!-- UR3e mounted on table -->
