Commit message: ur3e on table

File: urdf/ur3e_workcell.urdf.xacro (robot description, xacro)
@@ -2,14 +2,23 @@
 <robot xmlns:xacro="http://wiki.ros.org/xacro" name="ur3e_workcell">
   <xacro:include filename="$(find ur_description)/urdf/ur_macro.xacro"/>
+  <!-- World frame -->
   <link name="world"/>
+  <!-- Table mount point fixed in world -->
+  <link name="table_mount"/>
+  <joint name="world_to_table_mount" type="fixed">
+    <parent link="world"/>
+    <child link="table_mount"/>
+    <origin xyz="0.365 0.355 1.0" rpy="0 0 0"/>
+  </joint>
+  <!-- UR3e mounted on table -->
   <xacro:ur_robot
     name="ur3e"
     tf_prefix=""
-    parent="world"
+    parent="table_mount"
     joint_limits_parameters_file="$(find ur_description)/config/ur3e/joint_limits.yaml"
     kinematics_parameters_file="$(find ur_description)/config/ur3e/default_kinematics.yaml"
     physical_parameters_file="$(find ur_description)/config/ur3e/physical_parameters.yaml"
     visual_parameters_file="$(find ur_description)/config/ur3e/visual_parameters.yaml">
-    <origin xyz="0.19 0.39 1.0" rpy="0 0 0"/>
+    <origin xyz="0 0 0" rpy="0 0 0"/>
   </xacro:ur_robot>
 </robot>

Commit message: new gui for point selection

File: urdf/ur3e_workcell.urdf.xacro (robot description, xacro)
@@ -14,4 +14,18 @@
     <origin xyz="0.23 -0.03 0.724" rpy="0 0 0"/>
   </joint>
+  <!-- Trolley visual (shows in RViz; collision handled by planning_scene node) -->
+  <link name="trolley_link">
+    <visual>
+      <origin xyz="0 0 -0.041" rpy="0 0 0"/>
+      <geometry>
+        <mesh filename="package://fruitninja/meshes/UR3eTrolley.dae" scale="0.01 0.01 0.01"/>
+      </geometry>
+    </visual>
+  </link>
+  <joint name="world_to_trolley" type="fixed">
+    <parent link="world"/>
+    <child link="trolley_link"/>
+    <origin xyz="0 0 0" rpy="0 0 0"/>
+  </joint>
   <!-- UR3e mounted on table -->
   <xacro:ur_robot

Commit message: created grid system

File: urdf/ur3e_workcell.urdf.xacro (robot description, xacro)
@@ -17,5 +17,5 @@
   <link name="trolley_link">
     <visual>
-      <origin xyz="0 0 -0.041" rpy="0 0 0"/>
+      <origin xyz="0 0 0" rpy="1.5708 0 0"/>
       <geometry>
         <mesh filename="package://fruitninja/meshes/UR3eTrolley.dae" scale="0.01 0.01 0.01"/>
@@ -26,5 +26,5 @@
     <parent link="world"/>
     <child link="trolley_link"/>
-    <origin xyz="0 0 0" rpy="0 0 0"/>
+    <origin xyz="0.199 -0.13 0" rpy="1.5708 0 3.14159"/>
   </joint>
   <!-- UR3e mounted on table -->
